File: Dissatisfaction65.kicad_pcb (KiCad board)
At the start: 2 copper layers, 313.9 x 119.4 mm, 140 parts, among them SW1 Rotary_Encoder_Switch, SW2 SW_SPST, U1 Pro_Micro_ProMicro, U2 74HC4515, U3 SSD1306_I2C

Commit message: Placed NICE!-nano such that the micro usb comes right up to the edge of the board re-routed a bunch of column signals, the rotary encoder signals, reset switch, rotary encoder push button switch, 3v3, I2C signals, and gnd NICE!-nano should be encorporated now but should probably double check everything. DRC has two warnings about silkscreen getting clipped but there's nothing we can really do because the NICE-nano doesn't really fit anywhere else. Updated DRC constraints for JLCPCB fab. Should double check Added Circuit-Dude logo because I am circuit-dude and I did the layout and Thomas can't stop me unless he learns how to do layout.
Parts:
- added circuit-dude: LOGO, LOGO, F.Cu at (178.3, 118.1)
- Chico State Mechanical Keyboard Club: renamed from CMKC_LOGO
- moved U1 4.67 mm to (34.0, 44.0)
- moved Chico State Mechanical Keyboard Club 3.83 mm to (121.6, 119.3)
Connections:
- U1 pad 10: ENC_2 -> ENC_SW
- U1 pad 11: ENC_SW -> ENC_1
- U1 pad 12: unconnected-(U1-Pad12) -> ENC_2
- U1 pad 13: SDA -> SCL
- U1 pad 14: SCL -> SDA
- U1 pad 9: ENC_1 -> unconnected-(U1-Pad9)
Routing:
- net 3v3: track 28.5 -> 42.5 mm
- net ENC_1: track 278.8 -> 292.3 mm
- net ENC_2: track 267.9 -> 279.7 mm
- net ROW5: track 368.8 -> 380.3 mm
- net En: track 50.0 -> 61.5 mm
- net GND: track 415.9 -> 425.6 mm, vias 6 -> 3
- net ROW4: track 313.6 -> 322.1 mm, vias 2 -> 0
- net ROW2: track 283.6 -> 289.9 mm
- net ROW3: track 300.4 -> 306.4 mm, vias 2 -> 0
- net ROW1: track 277.0 -> 271.1 mm
- net ENC_SW: track 282.4 -> 286.4 mm
- net CLD1: track 16.7 -> 19.8 mm
- net E: track 28.2 -> 25.2 mm
- net CLD2: track 16.3 -> 19.3 mm
- net SDA: track 73.8 -> 71.0 mm
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